File: KiCad/senso v2/Senso V2.kicad_sch (KiCad schematic)
At the start: 17 parts

Commit message: update KiCad
Parts:
- added J1: PINHD_1x4_Female, Connector_PinSocket_2.54mm:PinSocket_1x04_P2.54mm_Vertical, symbol PCM_SL_Pin_Headers:PINHD_1x4_Female
- added J2: PINHD_1x4_Male, Connector_PinHeader_2.54mm:PinHeader_1x04_P2.54mm_Vertical, symbol PCM_SL_Pin_Headers:PINHD_1x4_Male
- renumbered D1 to LED_Blau, D4 to LED_Gelb, D3 to LED_Grün, D2 to LED_Rot
Connections:
- net at LED_Blau.1 (VSS): now also LED_Gelb.1 (VSS), LED_Grün.1 (VSS), LED_Rot.1 (VSS)
- net at LED_Blau.3 (VDD): now also LED_Gelb.3 (VDD), LED_Grün.3 (VDD), LED_Rot.3 (VDD)
- net at LED_Blau.4 (DOUT): now also LED_Gelb.2 (DIN)
- net at Taster_Rot_1.1, Taster_Rot_2.1: now also ESP32-PICO-V1.GND (Ground), Taster_Blau_1.1, Taster_Blau_2.1, Taster_Gelb_1.1, Taster_Gelb_2.1, Taster_Grün_1.1, Taster_Grün_2.1
- net at Taster_Rot_1.2, Taster_Rot_2.2: now also J2.2
- net at Taster_Grün_1.2, Taster_Grün_2.2: now also J2.1
- net at R5.1: now also ESP32-PICO-V1.25 (GPIO25)
- net at R5.2: now also J1.4
- net at R8.1: now also ESP32-PICO-V1.33 (GPIO33)
- net at R8.2: now also J1.1
- net at Taster_Gelb_1.2, Taster_Gelb_2.2: now also J2.3
- net at Taster_Blau_1.2, Taster_Blau_2.2: now also J2.4
- net at LED_Rot.2 (DIN): now also LED_Gelb.4 (DOUT)
- net at LED_Rot.4 (DOUT): now also LED_Grün.2 (DIN)
- net at ESP32-PICO-V1.26 (GPIO26): now also R6.1
- net at ESP32-PICO-V1.32 (GPIO32): now also R7.1
- net at R7.2: now also J1.2
- net at R6.2: now also J1.3
Other:
- moved on the sheet: LED_Blau, LED_Gelb, LED_Grün, LED_Rot, Taster_Blau_1, Taster_Blau_2, Taster_Gelb_1, Taster_Gelb_2, Taster_Grün_1, Taster_Grün_2, Taster_Rot_1, Taster_Rot_2
